File: Hardware/V1.2.0/LucaudioESP32_V1_2_0/LucaudiOptions.kicad_sch (KiCad schematic)
At the start: 13 parts, among them J1 Conn_01x04_Pin, J6 Conn_01x05_Pin, SW3 RotaryEncoder_Switch

Commit message: WIP
Connections:
- net GND: now also C31.2, C32.2
Changed lines of the file:
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@@
+	)
+	(junction
+		(at 48.26 113.03)
+		(diameter 0)
+		(color 0 0 0 0)
 	)
 	(junction
@@
 	(wire
 		(pts
+			(xy 48.26 113.03) (xy 49.53 113.03)
+		)
+		(stroke
+			(width 0)
+			(type default)
+		)
+	)
+	(wire
+		(pts
 			(xy 60.96 128.27) (xy 57.15 128.27)
 		)
@@
 	(wire
 		(pts
-			(xy 46.99 113.03) (xy 49.53 113.03)
+			(xy 46.99 113.03) (xy 48.26 113.03)
 		)
 		(stroke
@@
 	(symbol
 		(lib_id "power:GND")
+		(at 48.26 113.03 0)
+		(unit 1)
+		(exclude_from_sim no)
+		(in_bom yes)
+		(on_board yes)
+		(dnp no)
+		(fields_autoplaced yes)
+		(property "Reference" "#PWR09"
+			(at 48.26 119.38 0)
+			(effects
+				(font
+					(size 1.27 1.27)
+				)
+				(hide yes)
+			)
+		)
+		(property "Value" "GND"
+			(at 48.26 118.11 0)
+			(effects
+				(font
+					(size 1.27 1.27)
+				)
+			)
+		)
+		(property "Footprint" ""
+			(at 48.26 113.03 0)
+			(effects
+				(font
+					(size 1.27 1.27)
+				)
+				(hide yes)
+			)
+		)
+		(property "Datasheet" ""
+			(at 48.26 113.03 0)
+			(effects
+				(font
+					(size 1.27 1.27)
+				)
+				(hide yes)
+			)
+		)
+		(property "Description" "Power symbol creates a global label with name \"GND\" , ground"
+			(at 48.26 113.03 0)
+			(effects
+				(font
+					(size 1.27 1.27)
+				)
+				(hide yes)
+			)
+		)
+		(pin "1"
+		)
+		(instances
+			(project "LucaudioESP32_V1_2_0"
+				(path "/e38181f9-45f6-4f8a-b82f-a9fdcbe21bf2/73fd9b48-a15c-4c0e-bf10-cb7127373769"
+					(reference "#PWR09")
+					(unit 1)
+				)
+			)
+		)
+	)
+	(symbol
+		(lib_id "power:GND")
 		(at 53.34 151.13 0)
 		(unit 1)
@@
 		)
 		(instances
-			(project ""
+			(project "LucaudioESP32_V1_2_0"
 				(path "/e38181f9-45f6-4f8a-b82f-a9fdcbe21bf2/73fd9b48-a15c-4c0e-bf10-cb7127373769"
 					(reference "#PWR03")

Commit message: Update of V1.2.0
Parts:
- added Q1, Q2: BC847, Package_TO_SOT_SMD:SOT-23, symbol Transistor_BJT:BC847
- added R17, R18: 470, Resistor_SMD:R_0805_2012Metric_Pad1.20x1.40mm_HandSolder, symbol Device:R_Small
Connections:
- net 3V3_o: now also Q1.3 (C), Q2.3 (C)
- net LED_AMP_o: now also R18.2; no longer R10.2
- net LED_PWR_o: now also R17.2; no longer R13.2
- new net: Q2.1 (B), R17.1
- new net: Q1.2 (E), R10.2
- new net: Q1.1 (B), R18.1
- new net: Q2.2 (E), R13.2
Other:
- moved on the sheet: C31, C32, LED1, LED2, OLED1, R10, R13, R14, R5, R6, SW3
