File: Hardware/V1.2.0/LucaudioESP32_V1_2_0/LucaudioESP32_V1_2_0.kicad_pcb (KiCad board)
At the start: 2 copper layers, 92.4 x 70 mm, 88 parts, among them J1 Conn_01x04_Pin, J2 Conn_Coaxial_x2, J3 USB_C_Receptacle_USB2.0_16P, J4 Conn_01x04_Socket, J5 Conn_01x05_Socket, J6 Conn_01x05_Pin, J8 USB_B_Micro, J9 AudioJack3, SW1 SW_Omron_B3FS, SW2 SW_Omron_B3FS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

Commit message: WIP
Parts:
- removed the C31 at (156.3, 76.0)
- added C33: 100nF, Capacitor_SMD:C_0805_2012Metric, F.Cu at (156.3, 75.8)
- added OLED1: ~, local_lbr:OLED_128_32, F.Cu at (93.6, 130.4)
- added Q1: BC847, Package_TO_SOT_SMD:SOT-23, F.Cu at (92.5, 95.4)
- added Q2: BC847, Package_TO_SOT_SMD:SOT-23, F.Cu at (88.3, 95.4)
- added SW4: SW_SPDT, local_lbr:Slide_angular_SPDT, F.Cu at (137.0, 73.8)
- moved F1 0.98 mm to (156.0, 80.4)
Connections:
- C31 pad 2: Net-(C31-Pad2) -> GND
- C32 pad 2: Net-(C31-Pad2) -> GND
- F1 pad 1: Vusb -> Net-(SW4-B)
- R10 pad 2: LED_AMP_o -> Net-(Q1-E)
- R13 pad 2: LED_PWR_o -> Net-(Q2-E)
Routing:
- net 3V3_o: track 15.5 -> 42.8 mm
- net OLED_SCL: track 0.00 -> 23.7 mm
- net OLED_SDA: track 0.00 -> 19.5 mm
- net +5V: track 100.8 -> 96.0 mm
- net Vusb: track 22.7 -> 25.8 mm
- net GND: track 11.4 -> 12.8 mm, vias 123 -> 128
Other:
- outline, holes or cut-outs redrawn

Commit message: Update of V1.2.0
Parts:
- removed the REF** at (138.2, 74.0)
- added R17: 470, Resistor_SMD:R_0805_2012Metric_Pad1.20x1.40mm_HandSolder, B.Cu at (80.7, 98.2)
- added R18: 470, Resistor_SMD:R_0805_2012Metric_Pad1.20x1.40mm_HandSolder, B.Cu at (80.7, 95.6)
- J9: footprint Connector_JST:JST_EH_B3B-EH-A_1x03_P2.50mm_Vertical -> local_lbr:JST_3p_audio
- Q1, Q2, REF** (x3): moved to B.Cu
- moved F1 13.9 mm to (145.6, 71.2), turned to 0 degrees
- moved C33 11.0 mm to (145.6, 73.3), turned to 0 degrees
- moved R10 7.36 mm to (87.5, 92.9), turned to 0 degrees
- moved R13 6.87 mm to (87.5, 98.5), turned to 0 degrees
- moved Q2 6.07 mm to (87.5, 101.5), turned to 0 degrees
- moved Q1 5.03 mm to (87.5, 95.7), turned to 0 degrees
- moved SW4 3.30 mm to (136.0, 76.9)
- moved J9 2.54 mm to (155.6, 126.1)
- moved TP4 2.21 mm to (137.5, 82.8)
- turned REF** to 180 degrees (x3)
Connections:
- Q1 pad 1: LED_AMP_o -> Net-(Q1-B)
- Q2 pad 1: LED_PWR_o -> Net-(Q2-B)
Routing:
- net 3V3_o: track 42.8 -> 64.7 mm
- net +5V: track 96.0 -> 111.2 mm
- net Vusb: track 25.8 -> 40.1 mm, vias 0 -> 1
- net Net-(SW4-B): track 0.00 -> 12.6 mm
- net Net-(Q2-B): track 0.00 -> 7.57 mm
- net Net-(Q1-B): track 0.00 -> 5.37 mm
- net Net-(Q2-E): track 0.00 -> 3.58 mm
- net Net-(Q1-E): track 0.00 -> 3.45 mm
- net Net-(LED1-A): track 28.5 -> 31.2 mm
- net Net-(LED2-A): track 32.0 -> 34.6 mm
- net MCU_TX: track 31.5 -> 29.0 mm
- net MCU_RX: track 29.1 -> 28.0 mm
- net 3V3: track 143.6 -> 142.7 mm
- net ROTARY_B_o: track 29.8 -> 30.3 mm
- net GND: vias 128 -> 135
Other:
- board text added: "SN :"
