File: Hardware/V1.2.0/LucaudioESP32_V1_2_0/LucaudioESP32_V1_2_0.kicad_sch (KiCad schematic)
At the start: 65 parts, among them J2 Conn_Coaxial_x2, J3 USB_C_Receptacle_USB2.0_16P, J4 Conn_01x04_Socket, J5 Conn_01x05_Socket, J8 USB_B_Micro, J9 AudioJack3, SW1 SW_Omron_B3FS, SW2 SW_Omron_B3FS, U1 ESP32-WROVER-E, U2 LP5907MFX-3.3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

Commit message: WIP
Parts:
- added C33: 100nF, Capacitor_SMD:C_0805_2012Metric, symbol Device:C_Small
Connections:
- net GND: now also C33.2
- net Vusb: now also C33.1

Commit message: Update of V1.2.0
Parts:
- added SW4: SW_SPDT, local_lbr:Slide_angular_SPDT, symbol Switch:SW_SPDT
- J9: footprint Connector_JST:JST_EH_B3B-EH-A_1x03_P2.50mm_Vertical -> local_lbr:JST_3p_audio
Connections:
- net Vusb: now also SW4.1 (A); no longer C33.1, F1.1
- new net: C33.1, F1.1, SW4.2 (B)
Changed lines of the file:
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@@
 	)
 	(junction
-		(at 33.02 140.97)
-		(diameter 0)
-		(color 0 0 0 0)
-	)
-	(junction
 		(at 50.8 124.46)
 		(diameter 0)
@@
 	)
 	(junction
+		(at 33.02 140.97)
+		(diameter 0)
+		(color 0 0 0 0)
+	)
+	(junction
 		(at 38.1 124.46)
 		(diameter 0)
@@
 	(wire
 		(pts
-			(xy 29.21 140.97) (xy 33.02 140.97)
-		)
-		(stroke
-			(width 0)
-			(type default)
-		)
-	)
-	(wire
-		(pts
 			(xy 237.49 19.05) (xy 237.49 16.51)
 		)
@@
 	(wire
 		(pts
+			(xy 30.48 140.97) (xy 33.02 140.97)
+		)
+		(stroke
+			(width 0)
+			(type default)
+		)
+	)
+	(wire
+		(pts
 			(xy 113.03 142.24) (xy 113.03 147.32)
 		)
@@
 	(wire
 		(pts
+			(xy 19.05 143.51) (xy 20.32 143.51)
+		)
+		(stroke
+			(width 0)
+			(type default)
+		)
+	)
+	(wire
+		(pts
 			(xy 124.46 53.34) (xy 124.46 55.88)
 		)
@@
 	)
 	(rectangle
-		(start 123.19 17.78)
-		(end 139.7 22.86)
+		(start 149.352 15.621)
+		(end 165.862 20.701)
 		(stroke
 			(width 0)
@@
 		)
 	)
+	(text_box "Options"
+		(exclude_from_sim no)
+		(at 203.2 101.6 0)
+		(size 18.415 4.445)
+		(stroke
+			(width 0)
+			(type default)
+		)
+		(fill
+			(type none)
+		)
+		(effects
+			(font
+				(size 1.27 1.27)
+			)
+			(href "#2")
+		)
+	)
 	(text "PCM5102 DAC"
 		(exclude_from_sim no)
@@
 	(text "USB TO SERIAL"
 		(exclude_from_sim no)
-		(at 131.318 20.574 0)
+		(at 157.48 18.415 0)
 		(effects
 			(font
@@
 	(global_label "Vusb"
 		(shape output)
-		(at 29.21 140.97 180)
+		(at 19.05 143.51 180)
 		(fields_autoplaced yes)
 		(effects
@@
 		)
 		(property "Intersheetrefs" "${INTERSHEET_REFS}"
-			(at 21.8101 140.97 0)
+			(at 11.6501 143.51 0)
 			(effects
 				(font
@@
 	)
 	(symbol
+		(lib_id "Switch:SW_SPDT")
+		(at 25.4 140.97 180)
+		(unit 1)
+		(exclude_from_sim no)
+		(in_bom yes)
+		(on_board yes)
+		(dnp no)
+		(fields_autoplaced yes)
+		(property "Reference" "SW4"
+			(at 25.4 132.08 0)
+			(effects
+				(font
+					(size 1.27 1.27)
+				)
+			)
+		)
+		(property "Value" "SW_SPDT"
+			(at 25.4 134.62 0)
+			(effects
+				(font
+					(size 1.27 1.27)
+				)
+			)
+		)
+		(property "Footprint" "local_lbr:Slide_angular_SPDT"
+			(at 25.4 140.97 0)
+			(effects
+				(font
+					(size 1.27 1.27)
+				)
+				(hide yes)
+			)
+		)
+		(property "Datasheet" "~"
+			(at 25.4 133.35 0)
+			(effects
+				(font
+					(size 1.27 1.27)
+				)
+				(hide yes)
+			)
+		)
+		(property "Description" "Switch, single pole double throw"
+			(at 25.4 140.97 0)
+			(effects
+				(font
+					(size 1.27 1.27)
+				)
+				(hide yes)
+			)
+		)
+		(pin "1"
+		)
+		(pin "3"
+		)
+		(pin "2"
+		)
+		(instances
+			(project "LucaudioESP32_V1_2_0"
+				(path "/e38181f9-45f6-4f8a-b82f-a9fdcbe21bf2"
+					(reference "SW4")
+					(unit 1)
+				)
+			)
+		)
+	)
+	(symbol
 		(lib_id "Device:R_Small")
 		(at 50.8 171.45 180)
@@
 			)
 		)
-		(property "Footprint" "Connector_JST:JST_EH_B3B-EH-A_1x03_P2.50mm_Vertical"
+		(property "Footprint" "local_lbr:JST_3p_audio"
 			(at 177.8 123.19 0)
 			(effects
